File: pcb/chessbot.kicad_pcb (KiCad board)
At the start: 2 copper layers, 51 parts, among them J1 USB_C_ONLY_POWER, J2 Conn_01x03, J3 Conn_01x03, M1 Stepper_Motor_bipolar, M2 Stepper_Motor_bipolar, Q1 Q_NPN, Q2 Q_NPN, Q3 NMOS, SW1 SW_Push, SW2 SW_Push, U1 TMC2209_SILENTSTEPSTICK, U2 TMC2209_SILENTSTEPSTICK, U3 ESP32-WROOM-32D, U4 MP2393GTL-Z, U5 CH340C_C7464026, U6 GT-USB-7047B

Commit message: PCB routing
Parts:
- removed C15: 0.1uF, easyeda2kicad:C0603
- added C5: 0.1uF, easyeda2kicad:C0603, F.Cu at (111.4, 72.7)
- U1, U2: footprint TMC2209_SILENTSTEPSTICK:MODULE_TMC2209_SILENTSTEPSTICK -> TMC2209_SILENTSTEPSTICK:MODULE_TMC2209_SILENTSTEPSTICK_INTERNAL SILKSCREEN
- moved L1 159.7 mm to (184.8, 77.2), turned to 90 degrees
- moved D4 148.5 mm to (189.7, 76.4), turned to -90 degrees
- moved U1 139.9 mm to (170.9, 53.2), turned to -90 degrees
- moved R3 124.5 mm to (156.3, 80.5)
- moved U2 123.0 mm to (170.9, 70.5), turned to -90 degrees
- moved M1 113.8 mm to (184.8, 59.2), turned to 90 degrees
- moved M2 113.4 mm to (184.8, 70.2), turned to 90 degrees
- moved R15 110.9 mm to (143.2, 52.8), turned to 180 degrees
- moved C4 107.2 mm to (189.7, 72.7)
- moved R9 103.7 mm to (131.4, 48.8), turned to 90 degrees
- moved J2 102.8 mm to (174.9, 81.3)
- moved R11 102.0 mm to (135.6, 49.5), turned to -90 degrees
- moved R10 101.0 mm to (128.4, 51.0)
- moved R7 97.9 mm to (126.9, 49.5)
- moved R8 96.7 mm to (125.5, 51.0)
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Connections:
- C12 pad 1: Net-(C12-Pad1) -> BST
- C12 pad 2: BST -> Net-(C12-Pad2)
- C14 pad 1: Net-(C14-Pad1) -> GND
- C14 pad 2: DTR -> Net-(U5-V3)
- C3 pad 1: Net-(U5-V3) -> DTR
- C3 pad 2: GND -> Net-(C3-Pad2)
- C6 pad 1: 3V3 -> 12V
- C7 pad 1: 3V3 -> 12V
- M1 pad 1: 1_1A -> 1_2A
- M1 pad 2: 1_1B -> 1_1A
- M1 pad 3: 1_2A -> 1_1B
- M2 pad 1: 2_1A -> 2_2A
- M2 pad 2: 2_1B -> 2_1A
- M2 pad 3: 2_2A -> 2_1B
- R11 pad 1: Net-(C12-Pad1) -> Net-(C12-Pad2)
- R6 pad 1: Net-(C14-Pad1) -> Net-(C3-Pad2)
Routing:
- net 3V3: track 0.00 -> 148.8 mm, vias 0 -> 3
- net 12V: track 0.00 -> 118.3 mm
- net ESP-TMC: track 0.00 -> 114.0 mm
- net 2_DIR: track 0.00 -> 72.5 mm, vias 0 -> 1
- net 2_STEP: track 0.00 -> 69.5 mm, vias 0 -> 1
- net EN: track 0.00 -> 68.9 mm
- net 1_DIR: track 0.00 -> 59.8 mm, vias 0 -> 2
- net 1_STEP: track 0.00 -> 55.4 mm, vias 0 -> 2
- net EM: track 0.00 -> 51.7 mm, vias 0 -> 2
- net ENDSTOP1: track 0.00 -> 46.5 mm
- net ENDSTOP2: track 0.00 -> 35.8 mm
- net Net-(D4-A): track 0.00 -> 32.7 mm
- net USB-ESP: track 0.00 -> 28.6 mm
- net ESP-USB: track 0.00 -> 28.5 mm
- net IO: track 0.00 -> 24.9 mm
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- added copper zone on F.Cu, net 12V
- added copper zone on F.Cu, net 3V3
- added copper zone on B.Cu, net GND
- added copper zone on F.Cu, net GND
Other:
- board outline added: 100 x 41 mm
- board text added: "13kΩ"
- board text added: "40.2kΩ"
