File: pcb/chessbot.kicad_sch (KiCad schematic)
At the start: 48 parts, among them J1 USB_C_ONLY_POWER, M1 Stepper_Motor_bipolar, M2 Stepper_Motor_bipolar, Q1 Q_NPN, Q2 Q_NPN, Q3 NMOS, SW1 SW_Push, SW2 SW_Push, U1 TMC2209_SILENTSTEPSTICK, U2 TMC2209_SILENTSTEPSTICK, U3 ESP32-WROOM-32D, U4 MP2393GTL-Z, U5 CH340C_C7464026, U6 GT-USB-7047B

Commit message: Journal for yesterday: jlc component sourcing
Parts:
- removed C10: 47uF, symbol Device:C
- removed C7: 470uF, symbol Device:C_Polarized
- removed D1: SS14, Diode_SMD:D_SMA, symbol Diode:SS14
- removed Q1: Q_NPN, symbol Device:Q_NPN
- removed R14: 5.1kΩ, symbol Device:R_US
- removed R15: 1kΩ, symbol Device:R_US
- removed R2, R4, R5, R6: 10kΩ, symbol Device:R_US
- added C10, C16: 22uF, easyeda2kicad:C0805, symbol easyeda2kicad:CL21A226MAQNNNE
- added C7: 470uF, easyeda2kicad:CAP-SMD_BD10.0-L10.3-W10.3-FD, symbol easyeda2kicad:RVT1V471M1010
- added D4: SS14, easyeda2kicad:SMA_L4.2-W2.6-LS5.0-RD_1, symbol easyeda2kicad:SS14
- added J2, J3: Conn_01x03, Connector_JST:JST_PH_B3B-PH-K_1x03_P2.00mm_Vertical, symbol Connector_Generic:Conn_01x03
- added Q1: Q_NPN, easyeda2kicad:SOT-23-3_L2.9-W1.3-P1.90-LS2.4-BR, symbol easyeda2kicad:MMBT3904-C20526
- added R14: 5.1kΩ, easyeda2kicad:R0603, symbol easyeda2kicad:0603WAF5101T5E
- added R15: 1kΩ, easyeda2kicad:R0603, symbol easyeda2kicad:0603WAF1001T5E
- added R2, R4, R5, R6: 10kΩ, easyeda2kicad:R0805, symbol easyeda2kicad:0805W8F1002T5E
- C1, C14, C15, C3, C4, C9: footprint (none) -> easyeda2kicad:C0603; symbol Device:C -> easyeda2kicad:CC0603KRX7R9BB104; LCSC Part (none) -> C14663; MPN (none) -> CC0603KRX7R9BB104; Manufacturer (none) -> YAGEO(国巨)
- C11: value 7nF -> 6.8nF; footprint (none) -> easyeda2kicad:C0603; symbol Device:C -> easyeda2kicad:0603B682K500NT; LCSC Part (none) -> C1631; MPN (none) -> 0603B682K500NT; Manufacturer (none) -> FH(风华)
- C12: footprint (none) -> easyeda2kicad:C0603; symbol Device:C -> easyeda2kicad:CL10A105KB8NNNC; LCSC Part (none) -> C15849; MPN (none) -> CL10A105KB8NNNC; Manufacturer (none) -> SAMSUNG(三星)
- C13: footprint (none) -> easyeda2kicad:C0603; symbol Device:C -> easyeda2kicad:CL10C100JB8NNNC; LCSC Part (none) -> C1634; MPN (none) -> CL10C100JB8NNNC; Manufacturer (none) -> SAMSUNG(三星)
- C2: footprint (none) -> easyeda2kicad:C0603; symbol Device:C -> easyeda2kicad:CL10A106MA8NRNC; LCSC Part (none) -> C96446; MPN (none) -> CL10A106MA8NRNC; Manufacturer (none) -> SAMSUNG(三星)
- C6: footprint (none) -> easyeda2kicad:CAP-SMD_BD10.0-L10.3-W10.3-FD; symbol Device:C_Polarized -> easyeda2kicad:RVT1V471M1010; LCSC Part (none) -> C3350; MPN (none) -> RVT1V471M1010; Manufacturer (none) -> HONOR(荣誉)
- C8: footprint (none) -> easyeda2kicad:C0805; symbol Device:C -> easyeda2kicad:CL21A226MAQNNNE; LCSC Part (none) -> C45783; MPN (none) -> CL21A226MAQNNNE; Manufacturer (none) -> SAMSUNG(三星)
- D3: footprint (none) -> easyeda2kicad:LED0603-R-RD_AMBER; symbol Device:LED -> easyeda2kicad:BL-HJC36G-AV-TRB; LCSC Part (none) -> C165983; MPN (none) -> BL-HJC36G-AV-TRB; Manufacturer (none) -> BrtLed(佰鸿)
- J1, U1, U2: now left out of the parts list
- L1: footprint (none) -> Connector_JST:JST_PH_B2B-PH-K_1x02_P2.00mm_Vertical; now left out of the parts list
- L2: footprint (none) -> easyeda2kicad:L0805; symbol Device:L -> easyeda2kicad:CMI201209U2R2KT; LCSC Part (none) -> C1043; MPN (none) -> CMI201209U2R2KT; Manufacturer (none) -> FH(风华)
- M1, M2: footprint (none) -> Connector_JST:JST_PH_B4B-PH-K_1x04_P2.00mm_Vertical; now left out of the parts list
- Q2: footprint (none) -> easyeda2kicad:SOT-23-3_L2.9-W1.3-P1.90-LS2.4-BR; symbol Device:Q_NPN -> easyeda2kicad:MMBT3904-C20526; LCSC Part (none) -> C20526; MPN (none) -> MMBT3904(RANGE:100-300); Manufacturer (none) -> CJ(江苏长电/长晶)
- Q3: footprint (none) -> easyeda2kicad:SOT-23-3_L2.9-W1.3-P1.90-LS2.4-BR; symbol Simulation_SPICE:NMOS -> easyeda2kicad:AO3400A; LCSC Part (none) -> C20917; MPN (none) -> AO3400A; Manufacturer (none) -> AOS
- R1: footprint (none) -> easyeda2kicad:R0805; symbol Device:R_US -> easyeda2kicad:0805W8F1002T5E; LCSC Part (none) -> C17414; MPN (none) -> 0805W8F1002T5E; Manufacturer (none) -> UNI-ROYAL(厚声)
- R10: footprint (none) -> easyeda2kicad:R0603; symbol Device:R_US -> easyeda2kicad:0603WAF2202T5E; LCSC Part (none) -> C31850; MPN (none) -> 0603WAF2202T5E; Manufacturer (none) -> UNI-ROYAL(厚声)
- R11: footprint (none) -> easyeda2kicad:R0603; symbol Device:R_US -> easyeda2kicad:0603WAF200JT5E; LCSC Part (none) -> C22950; MPN (none) -> 0603WAF200JT5E; Manufacturer (none) -> UNI-ROYAL(厚声)
- R12: footprint (none) -> easyeda2kicad:R0603; symbol Device:R_US -> easyeda2kicad:0603WAF1001T5E; LCSC Part (none) -> C21190; MPN (none) -> 0603WAF1001T5E; Manufacturer (none) -> UNI-ROYAL(厚声)
- R13: footprint (none) -> easyeda2kicad:R0603; symbol Device:R_US -> easyeda2kicad:0603WAF5101T5E; LCSC Part (none) -> C23186; MPN (none) -> 0603WAF5101T5E; Manufacturer (none) -> UNI-ROYAL(厚声)
- R3: footprint (none) -> easyeda2kicad:R0603; symbol Device:R_US -> easyeda2kicad:0603WAF1000T5E; LCSC Part (none) -> C22775; MPN (none) -> 0603WAF1000T5E; Manufacturer (none) -> UNI-ROYAL(厚声)
- R7: footprint (none) -> easyeda2kicad:R0603; symbol Device:R_US -> easyeda2kicad:0603WAF4022T5E; LCSC Part (none) -> C12447; MPN (none) -> 0603WAF4022T5E; Manufacturer (none) -> UNI-ROYAL(厚声)
- R8: footprint (none) -> easyeda2kicad:R0603; symbol Device:R_US -> easyeda2kicad:0603WAF1302T5E; LCSC Part (none) -> C22797; MPN (none) -> 0603WAF1302T5E; Manufacturer (none) -> UNI-ROYAL(厚声)
- R9: value >300kΩ -> 560kΩ; footprint (none) -> easyeda2kicad:R0603; symbol Device:R_US -> easyeda2kicad:0603WAF5603T5E; LCSC Part (none) -> C23203; MPN (none) -> 0603WAF5603T5E; Manufacturer (none) -> UNI-ROYAL(厚声)
- SW1, SW2: footprint (none) -> Button_Switch_THT:SW_PUSH_6mm; now left out of the parts list
- U3: LCSC Part C473012 -> C529578
Connections:
- net 12V: now also C4.1, C8.1, C9.1, R9.2, D4.1 (K); no longer C4.2, C8.2, C9.2, R9.1
- net 3V3: now also C1.1, C13.1, C2.1, R1.2, R7.2, C10.2, C16.2, C7.1, J2.1 (Pin_1), J3.1 (Pin_1), R15.2, R2.2; no longer C1.2, C13.2, C2.2, R1.1, R7.1
- net BST: now also C12.2; no longer C12.1
- net DTR: now also C14.2; no longer C14.1
- net EM: now also R3.1; no longer R3.2
- net EN: now also R1.1, Q1.3 (C); no longer R1.2
- net EN_BUCK: now also R9.1; no longer R9.2
- net ESP-TMC: now also R12.1; no longer R12.2
- net FB: now also R10.2; no longer R10.1
- net GND: now also C1.2, C11.1, C2.2, C3.2, C4.2, C8.2, C9.2, D3.2 (C), Q2.2 (E), Q3.2 (S), R13.1, R8.1, U3.1 (GND), U3.15 (GND), U3.38 (GND), U3.39 (GND), C10.1, C16.1, C7.2, J2.3 (Pin_3), J3.3 (Pin_3), Q1.2 (E), R14.1, R4.2; no longer C1.1, C11.2, C2.1, C3.1, C4.1, C8.1, C9.1, D3.1 (K), Q2.E, Q3.3 (S), R13.2, R8.2
- net IO: now also Q2.3 (C), R2.1; no longer Q2.C
- net RTS: now also C15.2; no longer C15.1
- net SS: now also C11.2; no longer C11.1
- net SW: now also R11.2; no longer R11.1
- net at L1.1 (-): now also Q3.3 (D), D4.2 (A); no longer Q3.1 (D)
- net at U5.4 (V3): now also C3.1; no longer C3.2
- net at U3.28 (IO17): now also R12.2; no longer R12.1
- net ENDSTOP1: now reaches U3.36 (IO22)
- net ENDSTOP1: now also J2.2 (Pin_2)
- net ENDSTOP2: now reaches U3.37 (IO23)
- net ENDSTOP2: now also J3.2 (Pin_2)
- net at U6.A5 (CC1): now also R14.2
- net at U6.B5 (CC2): now also R13.2; no longer R13.1
- new net: C13.2, R10.1, R7.1, R8.2
- new net: Q3.1 (G), R3.2, R4.1
- new net: C15.1, R5.1
- new net: Q1.1 (B), R5.2
- new net: C12.1, R11.1
- new net: D3.1 (A), R15.1
- new net: C14.1, R6.1
- new net: Q2.1 (B), R6.2
- no-connect marks 14 -> 36
Other:
- moved on the sheet: SW2

Commit message: PCB routing
Parts:
- removed C15: 0.1uF, easyeda2kicad:C0603, symbol easyeda2kicad:CC0603KRX7R9BB104
- added C5: 0.1uF, easyeda2kicad:C0603, symbol easyeda2kicad:CC0603KRX7R9BB104
- C6, C7, D2, D3: now left out of the parts list
- Q1, Q2, Q3: FT Rotation Offset (none) -> 180
- U1, U2: footprint TMC2209_SILENTSTEPSTICK:MODULE_TMC2209_SILENTSTEPSTICK -> TMC2209_SILENTSTEPSTICK:MODULE_TMC2209_SILENTSTEPSTICK_INTERNAL SILKSCREEN
- U5: FT Rotation Offset (none) -> 90
Connections:
- net 12V: now also C6.1, C7.1
- net 1_1A: now also M1.2 (-); no longer M1.1
- net 1_1B: now also M1.3; no longer M1.2 (-)
- net 1_2A: now also M1.1; no longer M1.3
- net 2_1A: now also M2.2 (-); no longer M2.1
- net 2_1B: now also M2.3; no longer M2.2 (-)
- net 2_2A: now also M2.1; no longer M2.3
- net 3V3: no longer C6.1, C7.1
- net BST: now also C12.1; no longer C12.2
- net DTR: now also C3.1; no longer C14.2
- net GND: now also C14.1; no longer C3.2
- net RTS: now also C5.1
- net at R5.1: now also C5.2
- net at R11.1: now also C12.2; no longer C12.1
- net at U5.4 (V3): now also C14.2; no longer C3.1
- net at R6.1: now also C3.2; no longer C14.1
- net EN_TMC: no longer names the net of U1.16 (~{EN})
- net EN_TMC: no longer U2.16 (~{EN})
- no-connect marks 36 -> 38
Other:
- moved on the sheet: C12, C14, C3, R11
